File: pcb/test/test.kicad_pcb (KiCad board)
At the start: 2 copper layers, 17 parts, among them IC1 ADG904BRUZ-REEL7, J1 CONSMA013.062-G, J3 Conn_01x04, U2 TL081

Commit message: beaucoup vias
Parts:
- removed JP2: Jumper_2_Bridged, test_footprint_library:jumper20
- moved JP1 89.5 mm to (217.8, 88.7), turned to -135 degrees
- moved R1 29.2 mm to (229.9, 94.5), turned to 0 degrees
- moved C3 14.4 mm to (237.2, 77.1)
- moved U2 12.8 mm to (222.9, 89.1)
- moved R2 5.38 mm to (245.2, 88.6), turned to 90 degrees
- moved J3 2.80 mm to (226.0, 98.1)
Connections:
- IC1 pad 2: +2V5 -> Net-(IC1-VDD)
- J3 pad 1: +5V -> GND
- J3 pad 2: GND -> +5V
- J3 pad 3: Net-(J3-Pin_3) -> Net-(IC1-A1)
- J3 pad 4: Net-(J3-Pin_4) -> Net-(IC1-A0)
- JP1 pad 1: Net-(IC1-A1) -> +2V5
- JP1 pad 2: Net-(J3-Pin_4) -> Net-(IC1-VDD)
Routing:
- net Net-(IC1-A1): track 0.00 -> 89.6 mm
- net Net-(IC1-A0): track 0.00 -> 89.3 mm
- net GND: track 0.00 -> 85.7 mm, vias 0 -> 205
- net Net-(IC1-VDD): track 0.00 -> 78.8 mm
- net +5V: track 0.00 -> 33.9 mm
- net +2V5: track 0.00 -> 28.4 mm
- net Net-(U2-+): track 0.00 -> 24.5 mm
- added copper zone on B.Cu, net GND

Commit message: céfini
Connections:
- ANT1 pad 2: unconnected-(ANT1-NC-Pad2) -> GND
- ANT2 pad 2: unconnected-(ANT2-NC-Pad2) -> GND
- ANT3 pad 2: unconnected-(ANT3-NC-Pad2) -> GND
- ANT4 pad 2: unconnected-(ANT4-NC-Pad2) -> GND
Other:
- board outline added: 212 x 54 mm
Changed lines of the file:
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@@
 	(net 13 "Net-(IC1-RF3)")
 	(net 14 "Net-(IC1-RF4)")
-	(net 15 "unconnected-(ANT1-NC-Pad2)")
-	(net 16 "unconnected-(ANT2-NC-Pad2)")
-	(net 17 "unconnected-(ANT3-NC-Pad2)")
-	(net 18 "unconnected-(ANT4-NC-Pad2)")
-	(net 19 "Net-(IC1-VDD)")
+	(net 15 "Net-(IC1-VDD)")
 	(footprint "Resistor_SMD:R_0201_0603Metric"
 		(layer "F.Cu")
@@
 			(size 0.8 1.75)
 			(layers "F.Cu" "F.Paste" "F.Mask")
-			(net 18 "unconnected-(ANT4-NC-Pad2)")
+			(net 3 "GND")
 			(pinfunction "NC")
-			(pintype "no_connect")
+			(pintype "input")
 		)
 		(model "ST0147-00-011-A.stp"
@@
 			(size 0.8 1.75)
 			(layers "F.Cu" "F.Paste" "F.Mask")
-			(net 16 "unconnected-(ANT2-NC-Pad2)")
+			(net 3 "GND")
 			(pinfunction "NC")
-			(pintype "no_connect")
+			(pintype "input")
 		)
 		(model "ST0147-00-011-A.stp"
@@
 		(tags "Resistor Axial_DIN0411 series Axial Horizontal pin pitch 15.24mm 1W length 9.9mm diameter 3.6mm")
 		(property "Reference" "R1"
-			(at 7.62 -2.92 360)
+			(at 7.62 -2.92 0)
 			(layer "F.SilkS")
 			(effects
@@
 		)
 		(property "Value" "R"
-			(at 7.62 2.92 360)
+			(at 7.62 2.92 0)
 			(layer "F.Fab")
 			(effects
@@
 		)
 		(fp_text user "${REFERENCE}"
-			(at 7.62 0 360)
+			(at 7.62 0 0)
 			(layer "F.Fab")
 			(effects
@@
 			(size 0.8 1.75)
 			(layers "F.Cu" "F.Paste" "F.Mask")
-			(net 17 "unconnected-(ANT3-NC-Pad2)")
+			(net 3 "GND")
 			(pinfunction "NC")
-			(pintype "no_connect")
+			(pintype "input")
 		)
 		(model "ST0147-00-011-A.stp"
@@
 			(size 0.45 1.475)
 			(layers "F.Cu" "F.Paste" "F.Mask")
-			(net 19 "Net-(IC1-VDD)")
+			(net 15 "Net-(IC1-VDD)")
 			(pinfunction "VDD")
 			(pintype "passive")
@@
 			(size 0.8 1.75)
 			(layers "F.Cu" "F.Paste" "F.Mask")
-			(net 15 "unconnected-(ANT1-NC-Pad2)")
+			(net 3 "GND")
 			(pinfunction "NC")
-			(pintype "no_connect")
+			(pintype "input")
 		)
 		(model "ST0147-00-011-A.stp"
@@
 			(layers "*.Cu" "*.Mask")
 			(remove_unused_layers no)
-			(net 19 "Net-(IC1-VDD)")
+			(net 15 "Net-(IC1-VDD)")
 			(pinfunction "B")
 			(pintype "passive")
@@
 		)
 	)
+	(gr_line
+		(start 250.4 48.2)
+		(end 38.4 48.2)
+		(stroke
+			(width 0.05)
+			(type default)
+		)
+		(layer "Edge.Cuts")
+	)
+	(gr_line
+		(start 142.4 102.2)
+		(end 250.4 102.2)
+		(stroke
+			(width 0.05)
+			(type default)
+		)
+		(layer "Edge.Cuts")
+	)
+	(gr_line
+		(start 38.4 102.2)
+		(end 142.4 102.2)
+		(stroke
+			(width 0.05)
+			(type default)
+		)
+		(layer "Edge.Cuts")
+	)
+	(gr_line
+		(start 38.4 48.2)
+		(end 38.4 102.2)
+		(stroke
+			(width 0.05)
+			(type default)
+		)
+		(layer "Edge.Cuts")
+	)
+	(gr_line
+		(start 250.4 102.2)
+		(end 250.4 48.2)
+		(stroke
+			(width 0.05)
+			(type default)
+		)
+		(layer "Edge.Cuts")
+	)
 	(segment
 		(start 225.42 89.12)
@@
 		(width 0.2)
 		(layer "F.Cu")
-		(net 19)
+		(net 15)
 	)
 	(segment
@@
 		(width 0.2)
 		(layer "F.Cu")
-		(net 19)
+		(net 15)
 	)
 	(segment
@@
 		(width 0.2)
 		(layer "F.Cu")
-		(net 19)
+		(net 15)
 	)
 	(segment
@@
 		(width 0.2)
 		(layer "F.Cu")
-		(net 19)
+		(net 15)
 	)
 	(segment
@@
 		(width 0.2)
 		(layer "F.Cu")
-		(net 19)
+		(net 15)
 	)
 	(zone

Commit message: ajustement pour impression
Parts:
- removed JP1: Jumper_2_Bridged, test_footprint_library:jumper20
Connections:
- IC1 pad 2: Net-(IC1-VDD) -> +2V5
Routing:
- net +2V5: track 28.4 -> 122.1 mm, vias 0 -> 1
- net Net-(IC1-VDD): track 78.8 -> 0.00 mm
- net +5V: track 33.9 -> 35.4 mm
- net Net-(IC1-A1): track 89.6 -> 90.8 mm
Other:
- board text added: "ENSICAEN projet PERIPHERAL 08/01/2025 Antoine PICARD Paul JALLAIS Sara BOUSSOUF"

Commit message: pcb final
Routing:
- net +5V: track 35.4 -> 32.6 mm
- net Net-(U2-+): track 24.5 -> 26.5 mm
Other:
- board text added: "ENSICAEN projet PERIPHERAL 2024/2025 Antoine PICARD Paul JALLAIS Sara BOUSSOUF"
- board text removed: "ENSICAEN projet PERIPHERAL 08/01/2025 Antoine PICARD Paul JALLAIS Sara BOUSSOUF"
Changed lines of the file:
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@@
 		(layer "Edge.Cuts")
 	)
-	(gr_text "ENSICAEN\nprojet PERIPHERAL\n08/01/2025\n\nAntoine PICARD\nPaul JALLAIS\nSara BOUSSOUF"
-		(at 41.6 99.3 0)
+	(gr_text "ENSICAEN\nprojet PERIPHERAL\n2024/2025\n\nAntoine PICARD\nPaul JALLAIS\nSara BOUSSOUF"
+		(at 41.4 98 0)
 		(layer "F.Cu")
 		(effects
@@
 	)
 	(segment
+		(start 219.4 85.1)
+		(end 219.4 92.9)
+		(width 0.2)
+		(layer "F.Cu")
+		(net 2)
+	)
+	(segment
 		(start 223.5 98.085)
 		(end 223.46 98.125)
@@
 	)
 	(segment
-		(start 216 88.5)
-		(end 216 89.5)
+		(start 223.32 83.6)
+		(end 220.9 83.6)
+		(width 0.2)
+		(layer "F.Cu")
+		(net 2)
+	)
+	(segment
+		(start 219.4 92.9)
+		(end 221 94.5)
 		(width 0.2)
 		(layer "F.Cu")
@@
 	)
 	(segment
-		(start 223.92 83)
-		(end 221.5 83)
+		(start 225.42 81.5)
+		(end 223.32 83.6)
 		(width 0.2)
 		(layer "F.Cu")
@@
 	)
 	(segment
-		(start 225.42 81.5)
-		(end 223.92 83)
-		(width 0.2)
-		(layer "F.Cu")
-		(net 2)
-	)
-	(segment
-		(start 216 89.5)
-		(end 221 94.5)
-		(width 0.2)
-		(layer "F.Cu")
-		(net 2)
-	)
-	(segment
 		(start 221 94.5)
 		(end 229.88 94.5)
@@
 	)
 	(segment
-		(start 221.5 83)
-		(end 216 88.5)
+		(start 220.9 83.6)
+		(end 219.4 85.1)
 		(width 0.2)
 		(layer "F.Cu")
@@
 	)
 	(segment
-		(start 243.32 90.5)
-		(end 229.34 90.5)
+		(start 227.96 91.06)
+		(end 227.96 89.12)
+		(width 0.2)
+		(layer "F.Cu")
+		(net 7)
+	)
+	(segment
+		(start 242.32 91.5)
+		(end 228.4 91.5)
+		(width 0.2)
+		(layer "F.Cu")
+		(net 7)
+	)
+	(segment
+		(start 228.4 91.5)
+		(end 227.96 91.06)
 		(width 0.2)
 		(layer "F.Cu")
@@
 	)
 	(segment
-		(start 245.2 88.62)
-		(end 243.32 90.5)
-		(width 0.2)
-		(layer "F.Cu")
-		(net 7)
-	)
-	(segment
 		(start 245.12 94.5)
 		(end 245.12 88.7)
@@
 	)
 	(segment
-		(start 229.34 90.5)
-		(end 227.96 89.12)
-		(width 0.2)
-		(layer "F.Cu")
+		(start 245.2 88.62)
+		(end 242.32 91.5)
+		(width 0.2)
+		(layer "F.Cu")
